File: Board/p2mini-001.brd (EAGLE design)
At the start: 47 x 72 mm, 12 parts, among them K1 G5V-2, T1 2SC1815, U1 ARDUINO_PRO_MINI

Commit message: release
Parts:
- K1: value G5V-2 -> G5V1; device relay:G5V-2 -> relay:G5V1
- moved C1 26.2 mm to (12.7, 14.0)
- moved D1 15.5 mm to (33.0, 39.4)
- moved C2 14.9 mm to (12.7, 27.9)
- moved K1 4.02 mm to (22.9, 40.6)
- moved R1 3.59 mm to (10.2, 27.9)
- moved OK1 2.54 mm to (21.6, 26.7)
- moved JP1 2.54 mm to (5.08, 21.6)
- moved R3 2.54 mm to (10.2, 15.2)
Connections:
- removed net N$7: JP1.8, R3.2
- new net N$8: JP1.7, R3.2
- net GND: now also JP1.8; no longer K1.13
- net N$1: now also K1.10; no longer K1.8
- net N$2: now also K1.9; no longer K1.16
- net N$5: now also K1.5; no longer K1.4
- net N$6: now also U1.16; no longer K1.9
- net VCC: now also K1.2; no longer JP1.7, K1.1
Routing:
- net GND: track 111.8 -> 73.3 mm
- net VDD: track 94.6 -> 62.6 mm
- net N$6: track 46.5 -> 64.9 mm
- net MIDI1: track 30.6 -> 46.5 mm
- net N$7: track 13.4 -> 0.00 mm
- net N$8: track 0.00 -> 12.3 mm
- net N$13: track 19.8 -> 29.2 mm
- net N$1: track 37.7 -> 30.4 mm
- net N$5: track 25.6 -> 32.7 mm
- net VCC: track 83.2 -> 76.7 mm
- net RX: track 28.2 -> 23.1 mm
- net N$3: track 43.7 -> 46.6 mm
- net N$2: track 11.9 -> 14.2 mm
- net MIDI0: track 15.9 -> 14.9 mm
