File: Board/p2mini-001.sch (EAGLE design)
At the start: 12 parts, among them K1 G5V-2, T1 2SC1815, U1 ARDUINO_PRO_MINI

Commit message: release
Parts:
- K1: value G5V-2 -> G5V1; device relay:G5V-2 -> relay:G5V1
Connections:
- removed net N$7: JP1.8, R3.2
- new net N$8: JP1.7, R3.2
- net GND: now also JP1.8; no longer K12.P
- net N$1: now also K12.S; no longer K11.S
- net N$2: now also K11.2; no longer K1A.2
- net N$5: now also K12.P; no longer K11.P
- net N$6: now also U1.13; no longer K12.S
- net VCC: now also K11.1; no longer JP1.7, K1A.1
Other:
- moved on the sheet: C1, C2, R3
Changed lines of the file:
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@@
 <setting verticaltext="up"/>
 </settings>
-<grid distance="0.1" unitdist="inch" unit="inch" style="lines" multiple="1" display="yes" altdistance="0.01" altunitdist="inch" altunit="inch"/>
+<grid distance="0.1" unitdist="inch" unit="inch" style="lines" multiple="1" display="no" altdistance="0.01" altunitdist="inch" altunit="inch"/>
 <layers>
 <layer number="1" name="Top" color="4" fill="1" visible="no" active="no"/>
@@
 <part name="R2" library="resistor" deviceset="R-US_" device="0204/5" value="3k"/>
 <part name="D2" library="diode" deviceset="BAS15" device=""/>
-<part name="K1" library="relay" deviceset="G5V-2" device=""/>
 <part name="R3" library="resistor" deviceset="R-US_" device="0204/5" value="330"/>
 <part name="JP1" library="pinhead" deviceset="PINHD-1X8" device=""/>
 <part name="U1" library="SparkFun-Boards" deviceset="ARDUINO_PRO_MINI" device=""/>
+<part name="K1" library="relay" deviceset="G5V1" device=""/>
 </parts>
 <sheets>
 <sheet>
 <plain>
-<text x="215.9" y="-17.78" size="1.778" layer="91">Pineapple II Mini 0.0.0
+<text x="154.94" y="-17.78" size="1.778" layer="91">Pineapple II Mini 0.0.0
 Copyright 2015 by Pineapple.cc</text>
 <text x="215.9" y="25.4" size="1.778" layer="91">1: Vdd
@@
 <instance part="D1" gate="1" x="124.46" y="7.62"/>
 <instance part="VDD1" gate="G$1" x="93.98" y="60.96"/>
-<instance part="VDD2" gate="G$1" x="193.04" y="5.08"/>
-<instance part="SUPPLY4" gate="G$1" x="200.66" y="2.54"/>
-<instance part="SUPPLY5" gate="GND" x="200.66" y="-15.24"/>
-<instance part="SUPPLY3" gate="GND" x="193.04" y="-15.24"/>
-<instance part="C1" gate="G$1" x="193.04" y="-5.08"/>
-<instance part="C2" gate="G$1" x="200.66" y="-5.08"/>
+<instance part="VDD2" gate="G$1" x="208.28" y="5.08"/>
+<instance part="SUPPLY4" gate="G$1" x="215.9" y="2.54"/>
+<instance part="SUPPLY5" gate="GND" x="215.9" y="-15.24"/>
+<instance part="SUPPLY3" gate="GND" x="208.28" y="-15.24"/>
+<instance part="C1" gate="G$1" x="208.28" y="-5.08"/>
+<instance part="C2" gate="G$1" x="215.9" y="-5.08"/>
 <instance part="SUPPLY1" gate="GND" x="86.36" y="-15.24"/>
 <instance part="SUPPLY2" gate="G$1" x="88.9" y="53.34"/>
@@
 <instance part="R2" gate="G$1" x="139.7" y="17.78"/>
 <instance part="D2" gate="1" x="154.94" y="27.94" rot="R90"/>
-<instance part="K1" gate="A" x="162.56" y="27.94"/>
-<instance part="K1" gate="1" x="175.26" y="27.94" rot="R270"/>
-<instance part="K1" gate="2" x="175.26" y="10.16" rot="R270"/>
-<instance part="R3" gate="G$1" x="193.04" y="27.94"/>
+<instance part="R3" gate="G$1" x="193.04" y="48.26"/>
 <instance part="JP1" gate="A" x="210.82" y="35.56"/>
 <instance part="U1" gate="G$1" x="71.12" y="30.48"/>
+<instance part="K1" gate="1" x="162.56" y="27.94"/>
+<instance part="K1" gate="2" x="175.26" y="27.94" rot="R270"/>
 </instances>
 <busses>
@@
 <pinref part="C1" gate="G$1" pin="2"/>
 <pinref part="SUPPLY3" gate="GND" pin="GND"/>
-<wire x1="193.04" y1="-10.16" x2="193.04" y2="-12.7" width="0.1524" layer="91"/>
+<wire x1="208.28" y1="-10.16" x2="208.28" y2="-12.7" width="0.1524" layer="91"/>
 </segment>
 <segment>
 <pinref part="C2" gate="G$1" pin="2"/>
 <pinref part="SUPPLY5" gate="GND" pin="GND"/>
-<wire x1="200.66" y1="-10.16" x2="200.66" y2="-12.7" width="0.1524" layer="91"/>
+<wire x1="215.9" y1="-10.16" x2="215.9" y2="-12.7" width="0.1524" layer="91"/>
 </segment>
 <segment>
@@
 <wire x1="154.94" y1="-7.62" x2="86.36" y2="-7.62" width="0.1524" layer="91"/>
 <junction x="86.36" y="-7.62"/>
-<pinref part="K1" gate="2" pin="P"/>
-<wire x1="172.72" y1="10.16" x2="170.18" y2="10.16" width="0.1524" layer="91"/>
-<wire x1="170.18" y1="10.16" x2="170.18" y2="-7.62" width="0.1524" layer="91"/>
-<wire x1="170.18" y1="-7.62" x2="154.94" y2="-7.62" width="0.1524" layer="91"/>
-<junction x="154.94" y="-7.62"/>
 <pinref part="JP1" gate="A" pin="2"/>
 <pinref part="U1" gate="G$1" pin="GND@2"/>
+<pinref part="JP1" gate="A" pin="8"/>
+<wire x1="208.28" y1="27.94" x2="200.66" y2="27.94" width="0.1524" layer="91"/>
+<wire x1="200.66" y1="27.94" x2="200.66" y2="-7.62" width="0.1524" layer="91"/>
+<wire x1="200.66" y1="-7.62" x2="154.94" y2="-7.62" width="0.1524" layer="91"/>
+<junction x="154.94" y="-7.62"/>
 </segment>
 </net>
@@
 <pinref part="SUPPLY4" gate="G$1" pin="VCC"/>
 <pinref part="C2" gate="G$1" pin="1"/>
-<wire x1="200.66" y1="0" x2="200.66" y2="-2.54" width="0.1524" layer="91"/>
+<wire x1="215.9" y1="0" x2="215.9" y2="-2.54" width="0.1524" layer="91"/>
 </segment>
 <segment>
 <pinref part="SUPPLY2" gate="G$1" pin="VCC"/>
 <wire x1="83.82" y1="38.1" x2="88.9" y2="38.1" width="0.1524" layer="91"/>
-<wire x1="88.9" y1="38.1" x2="88.9" y2="48.26" width="0.1524" layer="91"/>
+<wire x1="88.9" y1="38.1" x2="88.9" y2="50.8" width="0.1524" layer="91"/>
 <pinref part="OK1" gate="A" pin="VE"/>
-<wire x1="88.9" y1="48.26" x2="88.9" y2="50.8" width="0.1524" layer="91"/>
 <wire x1="88.9" y1="2.54" x2="91.44" y2="2.54" width="0.1524" layer="91"/>
 <wire x1="88.9" y1="38.1" x2="88.9" y2="35.56" width="0.1524" layer="91"/>
@@
 <wire x1="154.94" y1="30.48" x2="154.94" y2="35.56" width="0.1524" layer="91"/>
 <junction x="154.94" y="35.56"/>
-<pinref part="K1" gate="A" pin="1"/>
-<pinref part="JP1" gate="A" pin="7"/>
-<wire x1="208.28" y1="30.48" x2="200.66" y2="30.48" width="0.1524" layer="91"/>
-<wire x1="200.66" y1="30.48" x2="200.66" y2="48.26" width="0.1524" layer="91"/>
-<wire x1="200.66" y1="48.26" x2="88.9" y2="48.26" width="0.1524" layer="91"/>
-<junction x="88.9" y="48.26"/>
 <pinref part="U1" gate="G$1" pin="VCC"/>
+<pinref part="K1" gate="1" pin="1"/>
 </segment>
 </net>
@@
 <pinref part="VDD2" gate="G$1" pin="VDD"/>
 <pinref part="C1" gate="G$1" pin="1"/>
-<wire x1="193.04" y1="2.54" x2="193.04" y2="-2.54" width="0.1524" layer="91"/>
+<wire x1="208.28" y1="2.54" x2="208.28" y2="-2.54" width="0.1524" layer="91"/>
 </segment>
 <segment>
@@
 <segment>
 <pinref part="OK1" gate="A" pin="VO"/>
-<label x="50.8" y="43.18" size="1.778" layer="95"/>
-<wire x1="50.8" y1="43.18" x2="60.96" y2="43.18" width="0.1524" layer="91"/>
-<wire x1="50.8" y1="5.08" x2="50.8" y2="43.18" width="0.1524" layer="91"/>
-<wire x1="91.44" y1="5.08" x2="50.8" y2="5.08" width="0.1524" layer="91"/>
+<wire x1="58.42" y1="43.18" x2="60.96" y2="43.18" width="0.1524" layer="91"/>
+<wire x1="58.42" y1="5.08" x2="58.42" y2="43.18" width="0.1524" layer="91"/>
+<wire x1="91.44" y1="5.08" x2="58.42" y2="5.08" width="0.1524" layer="91"/>
 <pinref part="U1" gate="G$1" pin="RXI"/>
 </segment>
@@
 <wire x1="154.94" y1="15.24" x2="154.94" y2="20.32" width="0.1524" layer="91"/>
 <junction x="154.94" y="20.32"/>
-<pinref part="K1" gate="A" pin="2"/>
+<pinref part="K1" gate="1" pin="2"/>
 </segment>
 </net>
@@
 <net name="N$1" class="0">
 <segment>
-<pinref part="K1" gate="1" pin="S"/>
 <wire x1="208.28" y1="35.56" x2="180.34" y2="35.56" width="0.1524" layer="91"/>
 <wire x1="180.34" y1="35.56" x2="180.34" y2="33.02" width="0.1524" layer="91"/>
 <pinref part="JP1" gate="A" pin="5"/>
+<pinref part="K1" gate="2" pin="S"/>
 </segment>
 </net>
 <net name="N$5" class="0">
 <segment>
-<pinref part="K1" gate="1" pin="P"/>
 <wire x1="172.72" y1="27.94" x2="170.18" y2="27.94" width="0.1524" layer="91"/>
 <wire x1="170.18" y1="27.94" x2="170.18" y2="20.32" width="0.1524" layer="91"/>
@@
 <wire x1="182.88" y1="33.02" x2="208.28" y2="33.02" width="0.1524" layer="91"/>
 <pinref part="JP1" gate="A" pin="6"/>
+<pinref part="K1" gate="2" pin="P"/>
 </segment>
 </net>
 <net name="N$6" class="0">
 <segment>
+<pinref part="U1" gate="G$1" pin="13"/>
+<wire x1="83.82" y1="25.4" x2="114.3" y2="25.4" width="0.1524" layer="91"/>
+<wire x1="114.3" y1="25.4" x2="114.3" y2="48.26" width="0.1524" layer="91"/>
 <pinref part="R3" gate="G$1" pin="1"/>
-<wire x1="187.96" y1="27.94" x2="185.42" y2="27.94" width="0.1524" layer="91"/>
-<wire x1="185.42" y1="27.94" x2="185.42" y2="17.78" width="0.1524" layer="91"/>
-<pinref part="K1" gate="2" pin="S"/>
-<wire x1="185.42" y1="17.78" x2="180.34" y2="17.78" width="0.1524" layer="91"/>
-<wire x1="180.34" y1="17.78" x2="180.34" y2="15.24" width="0.1524" layer="91"/>
-</segment>
-</net>
-<net name="N$7" class="0">
-<segment>
+<wire x1="187.96" y1="48.26" x2="114.3" y2="48.26" width="0.1524" layer="91"/>
+</segment>
+</net>
+<net name="N$8" class="0">
+<segment>
+<pinref part="JP1" gate="A" pin="7"/>
+<wire x1="208.28" y1="30.48" x2="200.66" y2="30.48" width="0.1524" layer="91"/>
+<wire x1="200.66" y1="30.48" x2="200.66" y2="48.26" width="0.1524" layer="91"/>
 <pinref part="R3" gate="G$1" pin="2"/>
-<pinref part="JP1" gate="A" pin="8"/>
-<wire x1="198.12" y1="27.94" x2="208.28" y2="27.94" width="0.1524" layer="91"/>
-</segment>
-</net>
+<wire x1="200.66" y1="48.26" x2="198.12" y2="48.26" width="0.1524" layer="91"/>
+</segment>
+</net>
